Commit message: Renamed occurrences of manta to urab_sub

File: descriptions/urab_sub_description/robots/urab_sub_default.xacro (robot description, xacro)
@@ -12,13 +12,13 @@
      limitations under the License.
 -->
-<robot name="manta" xmlns:xacro="http://www.ros.org/wiki/xacro" >
+<robot name="urab_sub" xmlns:xacro="http://www.ros.org/wiki/xacro" >
   <xacro:arg name="debug" default="0"/>
-  <xacro:arg name="namespace" default="manta"/>
+  <xacro:arg name="namespace" default="urab_sub"/>
   <xacro:arg name="inertial_reference_frame" default="world"/>
   <!-- Include the ROV macro file -->
-  <xacro:include filename="$(find urab_sub_description)/urdf/manta_base.xacro"/>
-  <xacro:include filename="$(find urab_sub_description)/urdf/manta_gazebo.xacro"/>
+  <xacro:include filename="$(find urab_sub_description)/urdf/urab_sub_base.xacro"/>
+  <xacro:include filename="$(find urab_sub_description)/urdf/urab_sub_gazebo.xacro"/>
   <!-- Create the rexrov -->
-  <xacro:manta_base
+  <xacro:urab_sub_base
     namespace="$(arg namespace)"
     inertial_reference_frame="$(arg inertial_reference_frame)">
@@ -31,8 +31,8 @@
         <debug>$(arg debug)</debug>
         <!-- Adding the hydrodynamic and hydrostatic parameters for the vehicle-->
-        <xacro:manta_hydro_model namespace="$(arg namespace)"/>
+        <xacro:urab_sub_hydro_model namespace="$(arg namespace)"/>
       </plugin>
     </gazebo>
-  </xacro:manta_base>
+  </xacro:urab_sub_base>
   <!-- Joint state publisher plugin -->
   <xacro:default_joint_state_publisher namespace="$(arg namespace)" update_rate="50"/>

File: descriptions/urab_sub_description/urdf/urab_sub_base.xacro (robot description, xacro)
@@ -47,7 +47,7 @@
   -->
   <!-- Parameters -->
-  <xacro:property name="namespace" value="manta"/>
-  <xacro:property name="visual_mesh_file" value="file://$(find urab_sub_description)/mesh/manta_shell.dae"/>
-  <xacro:macro name="manta_base" params="namespace *gazebo inertial_reference_frame">
+  <xacro:property name="namespace" value="urab_sub"/>
+  <xacro:property name="visual_mesh_file" value="file://$(find urab_sub_description)/mesh/urab_sub_shell.dae"/>
+  <xacro:macro name="urab_sub_base" params="namespace *gazebo inertial_reference_frame">
    <!-- Rigid body description of the base link -->
     <link name="${namespace}/base_link">
@@ -74,5 +74,5 @@
           </geometry>
         </visual>
-        <!-- In manta_base i've made collision planes to minize the GPU load -->
+        <!-- In urab_sub_base i've made collision planes to minize the GPU load -->
     <collision>
       <origin xyz="0 0 ${0}" rpy="0 0 0"/>
@@ -93,10 +93,10 @@
     receive topics on all its thrusters. The robot will not move just by launching
     this file alone -->
-  <xacro:include filename="$(find urab_sub_description)/urdf/manta_actuators.xacro"/>
+  <xacro:include filename="$(find urab_sub_description)/urdf/urab_sub_actuators.xacro"/>
    <!-- Publishes -->
    <!-- ONLY NEED FOR SIMULATIONS (GAZEBO SPECIFIC)
      This .xacro file has to run to be able to move the robot when controller
      commands have been sent to the thrusters-->
-  <xacro:include filename="$(find urab_sub_description)/urdf/manta_sensors.xacro"/>
+  <xacro:include filename="$(find urab_sub_description)/urdf/urab_sub_sensors.xacro"/>
   </xacro:macro>
   <gazebo reference="${namespace}/base_link">

File: descriptions/urab_sub_description/urdf/urab_sub_gazebo.xacro (robot description, xacro)
@@ -5,5 +5,5 @@
      Student2019 Manta AUV, Vortex NTNU. -->
 <robot xmlns:xacro="http://www.ros.org/wiki/xacro">
-  <xacro:macro name="manta_hydro_model" params="namespace">
+  <xacro:macro name="urab_sub_hydro_model" params="namespace">
     <!-- List of hydrodynamic models this robot's links -->
     <link name="${namespace}/base_link">
