Commit message: Gave sub the .stl file for visualization

File: descriptions/urab_sub_description/urdf/urab_sub_base.xacro (robot description, xacro)
@@ -48,5 +48,5 @@
   <!-- Parameters -->
   <xacro:property name="namespace" value="urab_sub"/>
-  <xacro:property name="visual_mesh_file" value="file://$(find urab_sub_description)/mesh/urab_sub_shell.dae"/>
+  <xacro:property name="visual_mesh_file" value="file://$(find urab_sub_description)/mesh/urab_sub.stl"/>
   <xacro:macro name="urab_sub_base" params="namespace *gazebo inertial_reference_frame">
    <!-- Rigid body description of the base link -->
@@ -69,7 +69,8 @@
         <!-- Code in rexrov2_base.xacro if use the flag use_simplified_mesh -->
         <visual>
-          <origin xyz="0 0 0" rpy="0 0 0"/>
+          <origin xyz="-0.22 0 0" rpy="1.5707 0 1.5707"/>
           <geometry>
-            <mesh filename="${visual_mesh_file}" scale="1 1 1" />
+            <!-- 1/15 * base = the simulated urab sub is 0.42 meters in width -->
+            <mesh filename="${visual_mesh_file}" scale="0.028 0.028 0.028" />
           </geometry>
         </visual>

Commit message: Changed some dimensions and configs

File: descriptions/urab_sub_description/urdf/urab_sub_base.xacro (robot description, xacro)
@@ -22,9 +22,9 @@
   -->
   <!-- Mass -->
-  <xacro:property name="mass" value="30.9"/>
+  <xacro:property name="mass" value="13"/>
   <!-- Describing the dimensions of the vehicle's bounding box: width, length, height -->
-  <xacro:property name="x_size" value="0.400"/>
-  <xacro:property name="y_size" value="0.400"/>
-  <xacro:property name="z_size" value="0.20066"/>
+  <xacro:property name="x_size" value="0.38449"/>
+  <xacro:property name="y_size" value="0.460"/>
+  <xacro:property name="z_size" value="0.286933"/>
   <!-- minion_usv_height is not really! It's just for run... We need first calculate the Fossen parameters -->
   <!-- Volume -->
